Commit message: refactor!: mechanical code-quality cleanup across the framework
Implements the mechanical scope of the framework code-quality umbrella:
module layout by ownership, facade and visibility cleanup, test ownership,
re-export removal, duplicate-helper consolidation, typed identifiers, dead
code, historical comments, and the automated gates for the rules that are
cheap to enforce.

Ownership and layout:
- api_tree.rs, runner.rs, handle.rs, webots_controller.rs and clock/scheduler
  split by responsibility into module directories; satellite modules that
  owned no concept folded into their owner.
- Every re-export ladder removed. Each public item has one canonical path;
  internal modules import from the owning module. The __private glob that
  leaked the whole participant module publicly is replaced by an explicit,
  documented macro ABI.
- Cross-module test buckets redistributed to the modules they test; the eight
  retired_* trybuild fixtures asserting deleted APIs stay deleted are gone.

Duplication:
- Timed<T> and its freshness gate, the capability lookup on Robot, the driver
  publish-rate schedule, angle and distance helpers, the drive target and
  localization predicates, and the encoder staleness horizon each have one
  owner now. DifferentialDrive gains a canonical home beside the kinematic
  config, with the forward and inverse relation on one type.
- KinematicConfig::drive_kinematics resolves every declared geometry through
  one reader; mecanum and Ackermann kinematics are implemented, and the
  omnidirectional variant states that the authored document carries no
  geometry to derive from.

Errors, panics and typing:
- ModelError, BusError, CompileError and the source vocabularies carry typed
  data instead of strings. anyhow is gone from phoxal-manifest's public API.
- Poisoned-lock expects on receive, logging and step paths now recover; the
  remaining panics are either removed by construction or carry a localized
  expect attribute naming the invariant.
- Validated newtypes replace raw String identifiers throughout the model,
  with byte-identical serialized form.

Tests:
- phoxal_model::RobotBuilder composes a validated Robot in memory, so a unit
  test states the robot it asserts on instead of loading a shared fixture and
  inheriting properties it never declared.
- fixture/ reduced to one robot declaring every component type; the variants
  that differed only by identity, wheel width or an unread role hint are gone.

Enforcement:
- workspace-policy gains a comment-reference rule rejecting issue and decision
  identifiers in committed comments, with fully qualified upstream references
  allowed. The ~150 existing violations are removed and the gate is enabled.

Also carries the SIGTERM handling that was already in the working tree,
preserved through the runner split as participant/runner/signal.rs.

Wire formats, topic keys, serialized shapes, the launch ABI and the authored
document grammar are unchanged. Architectural corrections remain out of scope.

File: fixture/robot/rgbd-imu-diff-drive/structure.urdf (robot description, URDF)
Before this commit: robot RgbdImuDiffDrive, 9 links, 8 joints
Links:
- added link gnss_mount
Joints:
- added joint gnss_mount_joint: type fixed, parent base_link, child gnss_mount, origin xyz=0 0 0.10 rpy=0 0 0
