Commit message: feat!: enforce revisioned map safety and robot footprints
Signed-off-by: phoxal-release-bot <release-bot@phoxal.com>

File: examples/hello-rover/components/wheel_drive/structure.urdf (robot description, URDF)
Before this commit: robot wheel_drive, 2 links, 1 joints
Links:
- link wheel: geometry visual cylinder length=0.03 radius=0.05

File: fixture/component/drive_motor/structure.urdf (robot description, URDF)
Before this commit: robot drive_motor_device, 2 links, 1 joints
Links:
- link rotor_link: geometry visual mesh filename=package://meshes/drive_motor.obj
